File: schematic/GPS-schematic.sch (KiCad schematic (older format))
At the start: 12 parts

Commit message: Various schematic additions, TODO list
Parts:
- removed DS?: Nokia5110LCD, symbol Nokia5110LCD
- added DS?: FPC-F10CBS00V0F, symbol FPC-F10CBS00V0F
- added P?: CONN_02X12, symbol CONN_02X12
- added PS?: AP3429/A, symbol AP3429/A
Connections:
- new net: DS?.1 (VDD0), P?.2 (P2)
- new net: DS?.10 (LDE-), P?.20 (P20)
- new net: DS?.11 (VSS), P?.22 (P22)
- new net: DS?.12 (VSS(NC)), P?.24 (P24)
- new net: DS?.2 (VDD1), P?.4 (P4)
- new net: DS?.3 (SI), P?.6 (P6)
- new net: DS?.4 (RSX), P?.8 (P8)
- new net: DS?.5 (CSX), P?.10 (P10)
- new net: DS?.6 (SCL), P?.12 (P12)
- new net: DS?.7 (VLCD), P?.14 (P14)
- new net: DS?.8 (RES), P?.16 (P16)
- new net: DS?.9 (LED+), P?.18 (P18)
Changed lines of the file:
@@
 LIBS:melexis
 LIBS:generic
+LIBS:diodesinc
+LIBS:GPS-schematic-cache
 EELAYER 25 0
 EELAYER END
@@
 F 3 "" H 2100 4750 60  0000 C CNN
 	1    2350 4700
-	1    0    0    -1
-$EndComp
-$Comp
-L Nokia5110LCD DS?
-U 1 1 5687720E
-P 5100 5000
-F 0 "DS?" H 5000 5250 60  0000 C CNN
-F 1 "Nokia5110LCD" H 5200 4750 60  0000 C CNN
-F 2 "" H 5100 4900 60  0000 C CNN
-F 3 "" H 5100 4900 60  0000 C CNN
-	1    5100 5000
 	1    0    0    -1
 $EndComp
@@
 	1    0    0    -1
 $EndComp
+$Comp
+L AP3429/A PS?
+U 1 1 56881270
+P 6050 2750
+F 0 "PS?" H 5950 3000 60  0000 C CNN
+F 1 "AP3429/A" H 6050 2600 60  0000 C CNN
+F 2 "" H 6050 2750 60  0000 C CNN
+F 3 "" H 6050 2750 60  0000 C CNN
+	1    6050 2750
+	1    0    0    -1
+$EndComp
+$Comp
+L FPC-F10CBS00V0F DS?
+U 1 1 56881CD8
+P 6300 4450
+F 0 "DS?" H 5800 4750 60  0000 C CNN
+F 1 "FPC-F10CBS00V0F" H 6450 4750 60  0000 C CNN
+F 2 "" H 6350 4450 60  0000 C CNN
+F 3 "" H 6350 4450 60  0000 C CNN
+	1    6300 4450
+	1    0    0    -1
+$EndComp
+$Comp
+L CONN_02X12 P?
+U 1 1 56881D97
+P 6300 5150
+F 0 "P?" H 6300 5800 50  0000 C CNN
+F 1 "CONN_02X12" V 6300 5150 50  0000 C CNN
+F 2 "" H 6300 3950 50  0000 C CNN
+F 3 "" H 6300 3950 50  0000 C CNN
+	1    6300 5150
+	0    -1   -1   0
+$EndComp
 $EndSCHEMATC
